File: HW2/me433_hw2.sch (EAGLE design)
At the start: 22 parts

Commit message: finished pcb and gerber files
Connections:
- net GND: no longer U$4.P$3
Changed lines of the file:
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@@
 <part name="U$4" library="slide_switch" deviceset="SLIDE_SWITCH" device=""/>
 <part name="P+2" library="supply1" deviceset="+5V" device=""/>
-<part name="GND15" library="supply1" deviceset="GND" device=""/>
 </parts>
 <sheets>
@@
 <instance part="U$4" gate="G$1" x="50.8" y="-48.26" rot="R180"/>
 <instance part="P+2" gate="1" x="50.8" y="-33.02"/>
-<instance part="GND15" gate="1" x="43.18" y="-33.02" rot="R180"/>
 </instances>
 <busses>
@@
 <wire x1="-20.32" y1="53.34" x2="-10.16" y2="53.34" width="0.1524" layer="91"/>
 </segment>
-<segment>
-<pinref part="U$4" gate="G$1" pin="P$3"/>
-<pinref part="GND15" gate="1" pin="GND"/>
-<wire x1="43.18" y1="-43.18" x2="43.18" y2="-35.56" width="0.1524" layer="91"/>
-</segment>
 </net>
